Commit message: Dwqdwq

File: robot_description/welding_support/urdf/weldingtable.xacro (robot description, xacro)
@@ -63,5 +63,5 @@
     <collision>
       <geometry>
-        <box size="0.8 1.0 0.02"/>
+        <box size="0.001 0.001 0.001"/>
       </geometry>
     </collision>

Commit message: delete all the pcd file

File: robot_description/welding_support/urdf/weldingtable.xacro (robot description, xacro)
@@ -5,10 +5,50 @@
   <xacro:ur3_robot prefix="" joint_limited="true"/>
   <xacro:include filename="$(find realsense2_description)/urdf/_d415.urdf.xacro" />
- <link name="world"/>
-  <joint name="world_to_robot" type="fixed">
+  <link name="bar2">
+    <visual>
+      <geometry>
+        <box size="0.8 0.04 0.04"/>
+      </geometry>
+      <material name="Steel">
+        <color rgba="0.5 0.5 0.5 1.0"/>
+      </material>
+    </visual>
+    <collision>
+      <geometry>
+        <box size="0.8 0.04 0.04"/>
+      </geometry>
+    </collision>
+  </link>
+  <link name="world"/>
+  <joint name="world_to_bar2" type="fixed">
     <parent link="world"/>
+    <child link="bar2"/>
+    <origin xyz="0 0.038 -0.02" rpy="0 0 0"/>
+  </joint>
+  <joint name="bar2_to_robot" type="fixed">
+    <parent link="bar2"/>
     <child link="base_link"/>
-    <origin xyz="0 0 0" rpy="0.0 0.0 0"/>
+    <origin xyz="0 -0.038 0.02" rpy="0.0 0.0 0"/>
    <!-- <origin xyz="-0.331 0.0 0.0079375" rpy="0.0 0.0 -1.5708"/>  -->
+  </joint>
+ <link name="bar1">
+    <visual>
+      <geometry>
+        <box size="0.8 0.04 0.04"/>
+      </geometry>
+      <material name="Steel">
+        <color rgba="0.5 0.5 0.5 1.0"/>
+      </material>
+    </visual>
+    <collision>
+      <geometry>
+        <box size="0.8 0.04 0.04"/>
+      </geometry>
+    </collision>
+  </link>
+  <joint name="bar2_to_bar1" type="fixed">
+    <parent link="bar2"/>
+    <child link="bar1"/>
+    <origin xyz="0 -0.08 0" rpy="0 0 0"/>
   </joint>
   <link name="table">
@@ -27,8 +67,8 @@
     </collision>
   </link>
-  <joint name="world_to_table" type="fixed">
-    <parent link="world"/>
+  <joint name="bar2_to_table" type="fixed">
+    <parent link="bar2"/>
     <child link="table"/>
-    <origin xyz="0.0 0.331 -0.0079375" rpy="0 0 0"/>
+    <origin xyz="0.0 0.35 -0.03" rpy="0 0 0"/>
   </joint>
   <sensor_d415 parent="tool0">

Commit message: 12.19

File: robot_description/welding_support/urdf/weldingtable.xacro (robot description, xacro)
@@ -5,50 +5,10 @@
   <xacro:ur3_robot prefix="" joint_limited="true"/>
   <xacro:include filename="$(find realsense2_description)/urdf/_d415.urdf.xacro" />
-  <link name="bar2">
-    <visual>
-      <geometry>
-        <box size="0.8 0.04 0.04"/>
-      </geometry>
-      <material name="Steel">
-        <color rgba="0.5 0.5 0.5 1.0"/>
-      </material>
-    </visual>
-    <collision>
-      <geometry>
-        <box size="0.8 0.04 0.04"/>
-      </geometry>
-    </collision>
-  </link>
-  <link name="world"/>
-  <joint name="world_to_bar2" type="fixed">
+ <link name="world"/>
+  <joint name="world_to_robot" type="fixed">
     <parent link="world"/>
-    <child link="bar2"/>
-    <origin xyz="0 0.038 -0.02" rpy="0 0 0"/>
-  </joint>
-  <joint name="bar2_to_robot" type="fixed">
-    <parent link="bar2"/>
     <child link="base_link"/>
-    <origin xyz="0 -0.038 0.02" rpy="0.0 0.0 0"/>
+    <origin xyz="0 0 0" rpy="0.0 0.0 0"/>
    <!-- <origin xyz="-0.331 0.0 0.0079375" rpy="0.0 0.0 -1.5708"/>  -->
-  </joint>
- <link name="bar1">
-    <visual>
-      <geometry>
-        <box size="0.8 0.04 0.04"/>
-      </geometry>
-      <material name="Steel">
-        <color rgba="0.5 0.5 0.5 1.0"/>
-      </material>
-    </visual>
-    <collision>
-      <geometry>
-        <box size="0.8 0.04 0.04"/>
-      </geometry>
-    </collision>
-  </link>
-  <joint name="bar2_to_bar1" type="fixed">
-    <parent link="bar2"/>
-    <child link="bar1"/>
-    <origin xyz="0 -0.08 0" rpy="0 0 0"/>
   </joint>
   <link name="table">
@@ -67,8 +27,8 @@
     </collision>
   </link>
-  <joint name="bar2_to_table" type="fixed">
-    <parent link="bar2"/>
+  <joint name="world_to_table" type="fixed">
+    <parent link="world"/>
     <child link="table"/>
-    <origin xyz="0.0 0.35 -0.03" rpy="0 0 0"/>
+    <origin xyz="0.0 0.331 -0.0079375" rpy="0 0 0"/>
   </joint>
   <sensor_d415 parent="tool0">

Commit message: calibration

File: robot_description/welding_support/urdf/weldingtable.xacro (robot description, xacro)
@@ -12,5 +12,4 @@
    <!-- <origin xyz="-0.331 0.0 0.0079375" rpy="0.0 0.0 -1.5708"/>  -->
   </joint>
- <!--
   <link name="table">
     <visual>
@@ -32,5 +31,5 @@
     <child link="table"/>
     <origin xyz="0.0 0.331 -0.0079375" rpy="0 0 0"/>
-  </joint>-->
+  </joint>
   <sensor_d415 parent="tool0">
     <origin xyz="0 -0.04 0.02" rpy="0 ${-pi/2} ${pi/2}"/>    <!-- origin xyz="0 -0.11 0.065 -->

Commit message: new ur driver passed

File: robot_description/welding_support/urdf/weldingtable.xacro (robot description, xacro)
@@ -2,6 +2,6 @@
 <robot name="weldingtable" xmlns:xacro="http://wiki.ros.org/xacro">
   <xacro:property name="pi" value="3.1415926535897931" />
-  <xacro:include filename="$(find ur_description)/urdf/ur3.urdf.xacro" />
-  <xacro:ur3_robot prefix="" joint_limited="true"/>
+  <xacro:include filename="$(find ur-description)/urdf/ur5.urdf.xacro" />
+  <xacro:ur5_robot prefix="" joint_limited="true"/>
   <xacro:include filename="$(find realsense2_description)/urdf/_d415.urdf.xacro" />
  <link name="world"/>
@@ -12,4 +12,5 @@
    <!-- <origin xyz="-0.331 0.0 0.0079375" rpy="0.0 0.0 -1.5708"/>  -->
   </joint>
+<!--
   <link name="table">
     <visual>
@@ -66,4 +67,5 @@
     <origin xyz="0 0.33 0.3785" rpy="0 0 -1.5708"/>
   </joint>
+-->
 <!--
   <sensor_d415 parent="world">
@@ -71,7 +73,10 @@
   </sensor_d415>
 -->
+<!--
   <sensor_d415 parent="tool0">
-    <origin xyz="0.01 -0.05 0.0282" rpy="0 ${-pi/2} ${pi/2}"/>    <!-- origin xyz="0 -0.11 0.065 -->
+    <origin xyz="0.01 -0.05 0.0282" rpy="0 ${-pi/2} ${pi/2}"/>     origin xyz="0 -0.11 0.065
   </sensor_d415>
+ -->
+<!--
     <link name="welding_torch">
       <visual>
@@ -94,3 +99,4 @@
     <origin xyz="0 0.055 0.29" rpy="0 0 0"/>
   </joint>
+-->
 </robot>

Commit message: Y-shape

File: robot_description/welding_support/urdf/weldingtable.xacro (robot description, xacro)
@@ -2,5 +2,5 @@
 <robot name="weldingtable" xmlns:xacro="http://wiki.ros.org/xacro">
   <xacro:property name="pi" value="3.1415926535897931" />
-  <xacro:include filename="$(find ur_description)/urdf/ur5.urdf.xacro" />
+  <xacro:include filename="$(find ur_description_)/urdf/ur5.urdf.xacro" />
   <xacro:ur5_robot prefix="" joint_limited="true"/>
   <xacro:include filename="$(find realsense2_description)/urdf/_d415.urdf.xacro" />
@@ -12,5 +12,4 @@
    <!-- <origin xyz="-0.331 0.0 0.0079375" rpy="0.0 0.0 -1.5708"/>  -->
   </joint>
-<!--
   <link name="table">
     <visual>
@@ -36,5 +35,5 @@
     <visual>
       <geometry>
-        <box size="0.05 0.05 1"/>
+        <box size="0.05 0.05 1.5"/>
       </geometry>
     </visual>
@@ -65,7 +64,6 @@
     <parent link="post"/>
     <child link="bar"/>
-    <origin xyz="0 0.33 0.3785" rpy="0 0 -1.5708"/>
+    <origin xyz="0 0.33 0.7785" rpy="0 0 -1.5708"/>
   </joint>
--->
 <!--
   <sensor_d415 parent="world">
@@ -73,10 +71,7 @@
   </sensor_d415>
 -->
-<!--
   <sensor_d415 parent="tool0">
-    <origin xyz="0.01 -0.05 0.0282" rpy="0 ${-pi/2} ${pi/2}"/>     origin xyz="0 -0.11 0.065
+    <origin xyz="0.0 -0.102 0.062" rpy="0 ${-pi/2} ${pi/2}"/> <!--  origin xyz="0 -0.11 0.065 -->
   </sensor_d415>
- -->
-<!--
     <link name="welding_torch">
       <visual>
@@ -85,4 +80,7 @@
         </geometry>
         <origin rpy="${pi/2} -0.84997 ${-pi/2}" xyz="0 0 0"/>
+      <material name="torch1">
+        <color rgba="0.1 0.1 0.5 1.0"/>
+      </material>
       </visual>
       <collision>
@@ -97,6 +95,28 @@
     <parent link="tool0"/>
     <child link="welding_torch"/>
-    <origin xyz="0 0.055 0.29" rpy="0 0 0"/>
+    <origin xyz="0 0.048 0.227" rpy="0 0 0"/>
   </joint>
--->
+    <link name="torchSupport">
+      <visual>
+        <geometry>
+          <mesh filename="package://welding_support/meshes/collision/torchSupport.STL" scale="0.001 0.001 0.001"/>
+        </geometry>
+        <origin rpy="0 0 0" xyz="0 0 0"/>
+      <material name="torchSupport1">
+        <color rgba="0.8 0.8 0.8 1.0"/>
+      </material>
+      </visual>
+      <collision>
+        <geometry>
+          <mesh filename="package://welding_support/meshes/collision/torchSupport.STL" scale="0.001 0.001 0.001"/>
+        </geometry>
+        <origin rpy="0 0 0" xyz="0 0 0"/>
+      </collision>
+      <origin xyz="0 0 0" rpy="0 0 0"/>
+    </link>
+  <joint name="torchSupport_to_tool0" type="fixed">
+    <parent link="tool0"/>
+    <child link="torchSupport"/>
+    <origin xyz="0.0325 0.0475 0.115" rpy="${-pi*3/2} ${-pi*3/2} ${-pi/2}"/>
+  </joint>
 </robot>
