Commit message: fix strange rotation for limit of UR3-urdf

File: robot_description/ur_description/urdf/ur3.urdf.xacro (robot description, xacro)
@@ -21,5 +21,5 @@
     wrist_1_lower_limit:=${-pi}    wrist_1_upper_limit:=${pi}
     wrist_2_lower_limit:=${-pi}    wrist_2_upper_limit:=${pi}
-    wrist_3_lower_limit:=${-pi}    wrist_3_upper_limit:=${pi}
+    wrist_3_lower_limit:=${0*pi}    wrist_3_upper_limit:=${2*pi}
     transmission_hw_interface:=hardware_interface/PositionJointInterface
     safety_limits:=false safety_pos_margin:=0.15

File: robot_description/welding_support/urdf/weldingtable.xacro (robot description, xacro)
@@ -5,45 +5,4 @@
   <xacro:ur3_robot prefix="" joint_limited="true"/>
   <xacro:include filename="$(find realsense2_description)/urdf/_d415.urdf.xacro" />
-  <link name="world"/>
-  <link name="table">
-    <visual>
-      <geometry>
-        <box size="0.8 1.0 0.02"/>
-      </geometry>
-      <material name="Wooden">
-        <color rgba="1.0 0.831 0.486 1.0"/>
-      </material>
-    </visual>
-    <collision>
-      <geometry>
-        <box size="1.0 1.0 0.015875"/>
-      </geometry>
-    </collision>
-  </link>
-  <joint name="world_to_table" type="fixed">
-    <parent link="world"/>
-    <child link="table"/>
-    <origin xyz="0.0 0.331 -0.0079375" rpy="0 0 0"/>
-  </joint>
-  <link name="bar1">
-    <visual>
-      <geometry>
-        <box size="0.8 0.04 0.04"/>
-      </geometry>
-      <material name="Steel">
-        <color rgba="0.5 0.5 0.5 1.0"/>
-      </material>
-    </visual>
-    <collision>
-      <geometry>
-        <box size="0.8 0.04 0.04"/>
-      </geometry>
-    </collision>
-  </link>
-  <joint name="table_to_bar1" type="fixed">
-    <parent link="table"/>
-    <child link="bar1"/>
-    <origin xyz="0 -0.45 0.03" rpy="0 0 0"/>
-  </joint>
   <link name="bar2">
     <visual>
@@ -61,14 +20,55 @@
     </collision>
   </link>
-  <joint name="table_to_bar2" type="fixed">
-    <parent link="table"/>
+  <link name="world"/>
+  <joint name="world_to_bar2" type="fixed">
+    <parent link="world"/>
     <child link="bar2"/>
-    <origin xyz="0 -0.37 0.03" rpy="0 0 0"/>
+    <origin xyz="0 0.038 -0.02" rpy="0 0 0"/>
   </joint>
-  <joint name="table_to_robot" type="fixed">
+  <joint name="bar2_to_robot" type="fixed">
     <parent link="bar2"/>
     <child link="base_link"/>
     <origin xyz="0 -0.038 0.02" rpy="0.0 0.0 0"/>
    <!-- <origin xyz="-0.331 0.0 0.0079375" rpy="0.0 0.0 -1.5708"/>  -->
+  </joint>
+ <link name="bar1">
+    <visual>
+      <geometry>
+        <box size="0.8 0.04 0.04"/>
+      </geometry>
+      <material name="Steel">
+        <color rgba="0.5 0.5 0.5 1.0"/>
+      </material>
+    </visual>
+    <collision>
+      <geometry>
+        <box size="0.8 0.04 0.04"/>
+      </geometry>
+    </collision>
+  </link>
+  <joint name="bar2_to_bar1" type="fixed">
+    <parent link="bar2"/>
+    <child link="bar1"/>
+    <origin xyz="0 -0.08 0" rpy="0 0 0"/>
+  </joint>
+  <link name="table">
+    <visual>
+      <geometry>
+        <box size="0.8 1.0 0.02"/>
+      </geometry>
+      <material name="Wooden">
+        <color rgba="1.0 0.831 0.486 1.0"/>
+      </material>
+    </visual>
+    <collision>
+      <geometry>
+        <box size="0.8 1.0 0.02"/>
+      </geometry>
+    </collision>
+  </link>
+  <joint name="bar2_to_table" type="fixed">
+    <parent link="bar2"/>
+    <child link="table"/>
+    <origin xyz="0.0 0.35 -0.03" rpy="0 0 0"/>
   </joint>
   <sensor_d415 parent="tool0">

Commit message: realtime

File: robot_description/ur_description/urdf/ur3.urdf.xacro (robot description, xacro)
@@ -330,5 +330,5 @@
     <link name="${prefix}tool0"/>
     <joint name="${prefix}wrist_3_link-tool0_fixed_joint" type="fixed">
-      <origin xyz="0 ${wrist_3_length} 0" rpy="${pi/-2.0} 0 0"/>
+      <origin xyz="0 ${wrist_3_length} 0" rpy="${pi/-2.0} ${pi} 0"/>
       <parent link="${prefix}wrist_3_link"/>
       <child link="${prefix}tool0"/>

Commit message: add vertical type

File: robot_description/ur_description/urdf/ur3.urdf.xacro (robot description, xacro)
@@ -330,5 +330,5 @@
     <link name="${prefix}tool0"/>
     <joint name="${prefix}wrist_3_link-tool0_fixed_joint" type="fixed">
-      <origin xyz="0 ${wrist_3_length} 0" rpy="${pi/-2.0} ${pi} 0"/>
+      <origin xyz="0 ${wrist_3_length} 0" rpy="${pi/-2.0} 0 0"/>
       <parent link="${prefix}wrist_3_link"/>
       <child link="${prefix}tool0"/>

File: robot_description/welding_support/urdf/weldingtable.xacro (robot description, xacro)
@@ -5,50 +5,10 @@
   <xacro:ur3_robot prefix="" joint_limited="true"/>
   <xacro:include filename="$(find realsense2_description)/urdf/_d415.urdf.xacro" />
-  <link name="bar2">
-    <visual>
-      <geometry>
-        <box size="0.8 0.04 0.04"/>
-      </geometry>
-      <material name="Steel">
-        <color rgba="0.5 0.5 0.5 1.0"/>
-      </material>
-    </visual>
-    <collision>
-      <geometry>
-        <box size="0.8 0.04 0.04"/>
-      </geometry>
-    </collision>
-  </link>
-  <link name="world"/>
-  <joint name="world_to_bar2" type="fixed">
+ <link name="world"/>
+  <joint name="world_to_robot" type="fixed">
     <parent link="world"/>
-    <child link="bar2"/>
-    <origin xyz="0 0.038 -0.02" rpy="0 0 0"/>
-  </joint>
-  <joint name="bar2_to_robot" type="fixed">
-    <parent link="bar2"/>
     <child link="base_link"/>
-    <origin xyz="0 -0.038 0.02" rpy="0.0 0.0 0"/>
+    <origin xyz="0 0 0" rpy="0.0 0.0 0"/>
    <!-- <origin xyz="-0.331 0.0 0.0079375" rpy="0.0 0.0 -1.5708"/>  -->
-  </joint>
- <link name="bar1">
-    <visual>
-      <geometry>
-        <box size="0.8 0.04 0.04"/>
-      </geometry>
-      <material name="Steel">
-        <color rgba="0.5 0.5 0.5 1.0"/>
-      </material>
-    </visual>
-    <collision>
-      <geometry>
-        <box size="0.8 0.04 0.04"/>
-      </geometry>
-    </collision>
-  </link>
-  <joint name="bar2_to_bar1" type="fixed">
-    <parent link="bar2"/>
-    <child link="bar1"/>
-    <origin xyz="0 -0.08 0" rpy="0 0 0"/>
   </joint>
   <link name="table">
@@ -67,8 +27,8 @@
     </collision>
   </link>
-  <joint name="bar2_to_table" type="fixed">
-    <parent link="bar2"/>
+  <joint name="world_to_table" type="fixed">
+    <parent link="world"/>
     <child link="table"/>
-    <origin xyz="0.0 0.35 -0.03" rpy="0 0 0"/>
+    <origin xyz="0.0 0.331 -0.0079375" rpy="0 0 0"/>
   </joint>
   <sensor_d415 parent="tool0">

Commit message: ar-marker

File: robot_description/ur_description/urdf/ur3.urdf.xacro (robot description, xacro)
@@ -330,5 +330,5 @@
     <link name="${prefix}tool0"/>
     <joint name="${prefix}wrist_3_link-tool0_fixed_joint" type="fixed">
-      <origin xyz="0 ${wrist_3_length} 0" rpy="${pi/-2.0} ${pi} 0"/>
+      <origin xyz="0 ${wrist_3_length} 0" rpy="${pi/-2.0} 0 0"/>    <!--rpy="${pi/-2.0} ${pi} 0 -->
       <parent link="${prefix}wrist_3_link"/>
       <child link="${prefix}tool0"/>

File: robot_description/welding_support/urdf/weldingtable.xacro (robot description, xacro)
@@ -12,4 +12,5 @@
    <!-- <origin xyz="-0.331 0.0 0.0079375" rpy="0.0 0.0 -1.5708"/>  -->
   </joint>
+ <!--
   <link name="table">
     <visual>
@@ -31,9 +32,9 @@
     <child link="table"/>
     <origin xyz="0.0 0.331 -0.0079375" rpy="0 0 0"/>
-  </joint>
+  </joint>-->
   <sensor_d415 parent="tool0">
-    <origin xyz="0 -0.11 0.065" rpy="0 ${-pi/2} ${pi/2}"/>
+    <origin xyz="0 -0.04 0.02" rpy="0 ${-pi/2} ${pi/2}"/>    <!-- origin xyz="0 -0.11 0.065 -->
   </sensor_d415>
-    <link name="welding_torch">
+   <!--  <link name="welding_torch">
       <visual>
         <geometry>
@@ -54,4 +55,4 @@
     <child link="welding_torch"/>
     <origin xyz="0 0.055 0.29" rpy="0 0 0"/>
-  </joint>
+  </joint> -->
 </robot>

Commit message: new camera layout

File: robot_description/ur_description/urdf/ur3.urdf.xacro (robot description, xacro)
@@ -330,5 +330,5 @@
     <link name="${prefix}tool0"/>
     <joint name="${prefix}wrist_3_link-tool0_fixed_joint" type="fixed">
-      <origin xyz="0 ${wrist_3_length} 0" rpy="${pi/-2.0} 0 0"/>    <!--rpy="${pi/-2.0} ${pi} 0 -->
+      <origin xyz="0 ${wrist_3_length} 0" rpy="${pi/-2.0} ${pi} 0"/>    <!--rpy="${pi/-2.0} ${pi} 0 -->
       <parent link="${prefix}wrist_3_link"/>
       <child link="${prefix}tool0"/>

File: robot_description/welding_support/urdf/weldingtable.xacro (robot description, xacro)
@@ -32,8 +32,42 @@
     <origin xyz="0.0 0.331 -0.0079375" rpy="0 0 0"/>
   </joint>
-  <sensor_d415 parent="tool0">
-    <origin xyz="0 -0.04 0.02" rpy="0 ${-pi/2} ${pi/2}"/>    <!-- origin xyz="0 -0.11 0.065 -->
+  <link name="post">
+    <visual>
+      <geometry>
+        <box size="0.05 0.05 1"/>
+      </geometry>
+    </visual>
+    <collision>
+      <geometry>
+        <box size="0.05 0.05 1"/>
+      </geometry>
+    </collision>
+  </link>
+  <joint name="table_to_post" type="fixed">
+    <parent link="table"/>
+    <child link="post"/>
+    <origin xyz="0 -0.525 0.5" rpy="0 0 0"/>
+  </joint>
+  <link name="bar">
+    <visual>
+      <geometry>
+        <box size="0.6 0.05 0.05"/>
+      </geometry>
+    </visual>
+    <collision>
+      <geometry>
+        <box size="0.7 0.05 0.05"/>
+      </geometry>
+    </collision>
+  </link>
+  <joint name="post_to_bar" type="fixed">
+    <parent link="post"/>
+    <child link="bar"/>
+    <origin xyz="0 0.33 0.3785" rpy="0 0 -1.5708"/>
+  </joint>
+  <sensor_d415 parent="world">
+    <origin xyz="0 0.443 0.8303" rpy="0 ${pi/2} ${pi/2}"/>    <!-- origin xyz="0 -0.11 0.065 -->
   </sensor_d415>
-   <!--  <link name="welding_torch">
+    <link name="welding_torch">
       <visual>
         <geometry>
@@ -54,4 +88,4 @@
     <child link="welding_torch"/>
     <origin xyz="0 0.055 0.29" rpy="0 0 0"/>
-  </joint> -->
+  </joint>
 </robot>

Commit message: start new algorithm

File: robot_description/ur_description/urdf/ur3.urdf.xacro (robot description, xacro)
@@ -330,5 +330,5 @@
     <link name="${prefix}tool0"/>
     <joint name="${prefix}wrist_3_link-tool0_fixed_joint" type="fixed">
-      <origin xyz="0 ${wrist_3_length} 0" rpy="${pi/-2.0} ${pi} 0"/>    <!--rpy="${pi/-2.0} ${pi} 0 -->
+      <origin xyz="0 ${wrist_3_length} 0" rpy="${pi/-2.0} 0 0"/>    <!--rpy="${pi/-2.0} ${pi} 0 || rpy="${pi/-2.0} ${pi} 0-->
       <parent link="${prefix}wrist_3_link"/>
       <child link="${prefix}tool0"/>

File: robot_description/welding_support/urdf/weldingtable.xacro (robot description, xacro)
@@ -66,7 +66,13 @@
     <origin xyz="0 0.33 0.3785" rpy="0 0 -1.5708"/>
   </joint>
+<!--
   <sensor_d415 parent="world">
-    <origin xyz="0 0.443 0.8303" rpy="0 ${pi/2} ${pi/2}"/>    <!-- origin xyz="0 -0.11 0.065 -->
+    <origin xyz="0 0.443 0.8303" rpy="0 ${pi/2} ${pi/2}"/>
   </sensor_d415>
+-->
+  <sensor_d415 parent="tool0">
+    <origin xyz="0.01 -0.05 0.0282" rpy="0 ${-pi/2} ${pi/2}"/>    <!-- origin xyz="0 -0.11 0.065 -->
+  </sensor_d415>
+<!--
     <link name="welding_torch">
       <visual>
@@ -89,3 +95,4 @@
     <origin xyz="0 0.055 0.29" rpy="0 0 0"/>
   </joint>
+-->
 </robot>
