Commit message: orientation graphical

File: weldingrobot/weldingrobot_description/weldingscene_description/urdf/weldingrobot.urdf.xacro (robot description, xacro)
@@ -14,5 +14,5 @@
     <visual>
       <geometry>
-        <box size="1 1 0.02"/>
+        <box size="1.5 1.5 0.02"/>
       </geometry>
       <material name="Wooden">
@@ -22,5 +22,5 @@
     <collision>
       <geometry>
-        <box size="1 1 0.02"/>
+        <box size="1.5 1.5 0.02"/>
       </geometry>
     </collision>
@@ -29,5 +29,5 @@
     <parent link="base_link"/>
     <child link="table"/>
-    <origin xyz="0 0.22 -0.01" rpy="0 0 0"/>
+    <origin xyz="0 0.4 -0.01" rpy="0 0 0"/>
   </joint>
   <link name="post">
@@ -46,5 +46,5 @@
     <parent link="table"/>
     <child link="post"/>
-    <origin xyz="0 -0.525 0.5" rpy="0 0 0"/>
+    <origin xyz="0 -0.725 0.5" rpy="0 0 0"/>
   </joint>
   <link name="bar">
@@ -68,4 +68,26 @@
     <origin xyz="0.0 -0.102 0.062" rpy="0 ${-pi/2} ${pi/2}"/>
   </sensor_d415>
+<!--
+   <link name="d415_cable">
+    <visual>
+      <geometry>
+        <box size="1.5 1.5 0.02"/>
+      </geometry>
+      <material name="Wooden">
+        <color rgba="0 0.0 0.1 1.0"/>
+      </material>
+    </visual>
+    <collision>
+      <geometry>
+        <box size="1.5 1.5 0.02"/>
+      </geometry>
+    </collision>
+  </link>
+  <joint name="tool0_to_d415_cable" type="fixed">
+    <parent link="tool0"/>
+    <child link="d415_cable"/>
+    <origin xyz="0 0.4 -0.01" rpy="0 0 0"/>
+  </joint>
+-->
     <!-- <link name="welding_torch">
       <visual>

Commit message: fully trajecotry 6DOF

File: weldingrobot/weldingrobot_description/weldingscene_description/urdf/weldingrobot.urdf.xacro (robot description, xacro)
@@ -115,5 +115,5 @@
           <mesh filename="package://weldingscene_description/meshes/collision/torch.stl" scale="0.001 0.001 0.001"/>
         </geometry>
-        <origin rpy="${pi/2} -0.84997 ${-pi/2}" xyz="0 0 0"/>
+        <origin rpy="${pi/2} 0 ${-pi/2}" xyz="0 0 0"/>
       <material name="torch1">
         <color rgba="0.1 0.1 0.5 1.0"/>
@@ -124,5 +124,5 @@
           <mesh filename="package://weldingscene_description/meshes/collision/torch.stl" scale="0.001 0.001 0.001"/>
         </geometry>
-        <origin rpy="${pi/2} -0.84997 ${-pi/2}" xyz="0 0 0"/>
+        <origin rpy="${pi/2} 0 ${-pi/2}" xyz="0 0 0"/>
       </collision>
     </link>
@@ -130,5 +130,5 @@
       <parent link="tool0"/>
       <child link="welding_torch"/>
-      <origin xyz="0 0.048 0.227" rpy="0 0 0"/>
+      <origin xyz="0 0.048 0.227" rpy="-0.84997 0 0"/>
     </joint>
     <link name="torchSupport">
