Commit message: final

File: weldingrobot_config/weldingrobot_description/weldingscene_description/urdf/weldingrobot.urdf.xacro (robot description, xacro)
@@ -5,6 +5,4 @@
   <xacro:ur5_robot prefix="" joint_limited="true"/>
   <xacro:include filename="$(find realsense2_description)/urdf/_d415.urdf.xacro" />
-  <xacro:include filename="$(find kinect2_description)/urdf/kinect2_urdf.xacro" />
-  <xacro:kinect2 prefix=""/>
  <link name="world"/>
   <joint name="world_to_robot" type="fixed">
@@ -13,114 +11,7 @@
     <origin xyz="0 0 0" rpy="0.0 0.0 0"/>
   </joint>
-  <link name="table">
-    <visual>
-      <geometry>
-        <box size="1.5 1.5 0.02"/>
-      </geometry>
-      <material name="Wooden">
-        <color rgba="1.0 0.831 0.486 1.0"/>
-      </material>
-    </visual>
-    <collision>
-      <geometry>
-        <box size="1.5 1.5 0.02"/>
-      </geometry>
-    </collision>
-  </link>
-  <joint name="base_link_to_table" type="fixed">
-    <parent link="base_link"/>
-    <child link="table"/>
-    <origin xyz="0 0.4 -0.01" rpy="0 0 0"/>
-  </joint>
-  <link name="post">
-    <visual>
-      <geometry>
-        <box size="0.05 0.05 1.5"/>
-      </geometry>
-    </visual>
-    <collision>
-      <geometry>
-        <box size="0.05 0.05 1.5"/>
-      </geometry>
-    </collision>
-  </link>
-  <joint name="table_to_post" type="fixed">
-    <parent link="table"/>
-    <child link="post"/>
-    <origin xyz="0 -0.725 0.5" rpy="0 0 0"/>
-  </joint>
-  <link name="bar">
-    <visual>
-      <geometry>
-        <box size="0.6 0.05 0.05"/>
-      </geometry>
-    </visual>
-    <collision>
-      <geometry>
-        <box size="0.6 0.05 0.05"/>
-      </geometry>
-    </collision>
-  </link>
-  <joint name="post_to_bar" type="fixed">
-    <parent link="post"/>
-    <child link="bar"/>
-    <origin xyz="0 0.33 0.7785" rpy="0 0 -1.5708"/>
-  </joint>
-  <link name="kinect2_rgb_optical_frame"/>
-  <joint name="rgb_optical_frame" type="fixed">
-    <origin xyz="0 0 0" rpy="0 0 0"/>
-    <parent link="kinect2_link"/>
-    <child link="kinect2_rgb_optical_frame"/>
-  </joint>
-  <joint name="world_to_camera" type="fixed">
-    <parent link="world"/>
-    <child link="kinect2_link"/>
-    <origin xyz="0.1 0.43 1.2" rpy="0 3.14159 3.14159"/>
-  </joint>
   <sensor_d415 parent="tool0">
-    <origin xyz="0.0 -0.102 0.062" rpy="0 ${-pi/2} ${pi/2}"/>
+    <origin xyz="1.0 -0.102 0.062" rpy="0 ${-pi/2} ${pi/2}"/>
   </sensor_d415>
-<!--
-   <link name="d415_cable">
-    <visual>
-      <geometry>
-        <box size="1.5 1.5 0.02"/>
-      </geometry>
-      <material name="Wooden">
-        <color rgba="0 0.0 0.1 1.0"/>
-      </material>
-    </visual>
-    <collision>
-      <geometry>
-        <box size="1.5 1.5 0.02"/>
-      </geometry>
-    </collision>
-  </link>
-  <joint name="tool0_to_d415_cable" type="fixed">
-    <parent link="tool0"/>
-    <child link="d415_cable"/>
-    <origin xyz="0 0.4 -0.01" rpy="0 0 0"/>
-  </joint>
--->
-    <!-- <link name="welding_torch">
-      <visual>
-        <geometry>
-          <mesh filename="package://weldingscene_description/meshes/collision/torch.stl" scale="0.001 0.001 0.001"/>
-        </geometry>
-      <material name="torch1">
-        <color rgba="0.1 0.1 0.5 1.0"/>
-      </material>
-      </visual>
-      <collision>
-        <geometry>
-          <mesh filename="package://weldingscene_description/meshes/collision/torch.stl" scale="0.001 0.001 0.001"/>
-        </geometry>
-      </collision>
-    </link>
-  <joint name="torch_to_tool0" type="fixed">
-    <parent link="tool0"/>
-    <child link="welding_torch"/>
-    <origin xyz="0 0.035 0.234" rpy="${pi/2} ${-pi/4} ${-pi/2}"/>
-  </joint>  -->
     <link name="welding_torch">
       <visual>
@@ -143,5 +34,5 @@
       <parent link="tool0"/>
       <child link="welding_torch"/>
-      <origin xyz="0 0.048 0.227" rpy="-0.84997 0 0"/>
+      <origin xyz="1 0.048 0.227" rpy="-0.84997 0 0"/>
     </joint>
     <link name="torchSupport">
@@ -163,5 +54,5 @@
     <parent link="tool0"/>
     <child link="torchSupport"/>
-    <origin xyz="0.0325 0.0475 0.115" rpy="${-pi*3/2} ${-pi*3/2} ${-pi/2}"/>
+    <origin xyz="1.0325 0.1275 0.115" rpy="${-pi*3/2} ${-pi*3/2} ${-pi/2}"/>
   </joint>
 </robot>
